File: test_!/test_!.kicad_pcb (KiCad board)
At the start: 2 copper layers, 45 parts, among them J1 Screw_Terminal_01x02, SW1 SW_Push, SW2 SW_Wuerth_450301014042, U1 LM2574N-5, U2 NE555P, U4 4027, U5 4027, U6 74LS47, U7 HDSP-7401

Commit message: test
Parts:
- U3: footprint Package_DIP:DIP-16_W7.62mm_Socket_LongPads -> Package_TO_SOT_SMD:SOT-23-6
- U5: footprint Display_7Segment:HDSP-7401 -> Package_DIP:DIP-16_W7.62mm_Socket_LongPads
- U6: footprint Package_TO_SOT_SMD:SOT-23-6 -> Package_DIP:DIP-16_W7.62mm_Socket_LongPads
- moved H1 157.4 mm to (258.0, 115.9)
- moved H2 157.4 mm to (258.0, 128.4)
- moved H3 157.4 mm to (258.0, 141.0)
- moved H4 157.4 mm to (258.0, 153.6)
- moved D2 154.5 mm to (263.0, 24.0), turned to -90 degrees
- moved D3 150.5 mm to (255.5, 24.0), turned to -90 degrees
- moved D4 147.3 mm to (248.1, 24.0), turned to -90 degrees
- moved D5 144.7 mm to (240.6, 24.0), turned to -90 degrees
- moved R19 139.1 mm to (45.7, 149.0), turned to 90 degrees
- moved R20 134.5 mm to (49.0, 149.0), turned to 90 degrees
- moved C3 130.4 mm to (46.8, 177.0), turned to 90 degrees
- moved U2 126.2 mm to (45.2, 165.8), turned to 90 degrees
- moved C4 125.8 mm to (50.2, 177.0), turned to 90 degrees
- moved R1 125.1 mm to (256.1, 34.0), turned to -90 degrees
- moved R2 123.5 mm to (252.1, 34.0), turned to -90 degrees
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Other:
- board outline added: 100 x 80 mm

Commit message: test
tewtw
Parts:
- SW2: footprint Button_Switch_SMD:Nidec_Copal_CAS-120A -> Button_Switch_THT:SW_Slide_SPDT_Straight_CK_OS102011MS2Q
- moved H1 170.8 mm to (101.5, 47.5)
- moved H3 160.1 mm to (100.5, 112.5)
- moved SW1 107.5 mm to (140.2, 109.8), turned to -90 degrees
- moved H2 107.3 mm to (187.5, 47.5)
- moved U2 105.8 mm to (106.7, 79.7), turned to 0 degrees
- moved C3 102.3 mm to (98.9, 89.0), turned to 0 degrees
- moved D5 97.7 mm to (150.0, 60.5), turned to 90 degrees
- moved D4 97.7 mm to (157.5, 60.5), turned to 90 degrees
- moved D2 97.7 mm to (172.4, 60.5), turned to 90 degrees
- moved D3 97.7 mm to (165.0, 60.5), turned to 90 degrees
- moved C4 97.6 mm to (99.1, 92.5), turned to 180 degrees
- moved R4 94.7 mm to (150.0, 45.5)
- moved R3 91.3 mm to (157.5, 45.5)
- moved L1 90.8 mm to (133.0, 62.0), turned to 0 degrees
- moved R19 88.5 mm to (99.2, 78.5), turned to 180 degrees
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Routing:
- net GND: track 0.00 -> 265.7 mm, vias 0 -> 1
- net +5V: track 0.00 -> 164.1 mm
- net Clock: track 0.00 -> 40.7 mm, vias 0 -> 1
- net Net-(SW2-A): track 0.00 -> 36.0 mm
- net Net-(U2-THR): track 0.00 -> 35.5 mm, vias 0 -> 1
- net Net-(D1-K): track 0.00 -> 33.6 mm, vias 0 -> 1
- net VDD: track 0.00 -> 32.6 mm
- net Net-(U7-B): track 0.00 -> 30.4 mm
- net 555: track 0.00 -> 23.3 mm
- net Net-(U7-A): track 0.00 -> 18.7 mm
- net (no net): track 0.00 -> 18.3 mm, vias 0 -> 1
- net Net-(R13-Pad1): track 0.00 -> 10.6 mm
- net Net-(U2-DIS): track 0.00 -> 5.55 mm
- net Net-(D4-A): track 0.00 -> 4.88 mm
- net Net-(D5-A): track 0.00 -> 4.84 mm
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
Commit message: testes
adadada
Routing:
- net GND: track 265.7 -> 473.2 mm
- net Q2: track 0.00 -> 167.4 mm, vias 0 -> 2
- net +5V: track 164.1 -> 319.0 mm, vias 0 -> 3
- net Q1: track 0.00 -> 124.9 mm, vias 0 -> 1
- net Net-(U5B-J): track 0.00 -> 84.9 mm, vias 0 -> 1
- net QO: track 0.00 -> 82.8 mm, vias 0 -> 1
- net Q3: track 0.00 -> 78.4 mm
- net RESET: track 0.00 -> 43.1 mm
- net Net-(U7-G): track 0.00 -> 38.7 mm
- net Net-(U7-E): track 0.00 -> 35.4 mm
- net Net-(U6-BI): track 0.00 -> 34.6 mm
- net Net-(U5A-J): track 0.00 -> 33.5 mm
- net Net-(U4A-J): track 0.00 -> 28.5 mm, vias 0 -> 1
- net Net-(U7-F): track 0.00 -> 27.8 mm, vias 0 -> 1
- net Net-(U7-D): track 0.00 -> 26.3 mm
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